Commit message: feat: add dummy tool description

File: peeks_robot_descriptions/urdf/inc/common.xacro (robot description, xacro)
@@ -1,7 +1,7 @@
 <?xml version="1.0"?>
 <robot xmlns:xacro="http://wiki.ros.org/xacro">
-  <!-- 从指定型号的yaml文件中加载配置数据。 -->
+  <!-- 从yaml文件中加载机器人配置数据。 -->
   <xacro:macro
-    name="read_model_config"
+    name="read_robot_config"
     params="joint_limit_parameter_file
             robot_kinematics_parameter_file
@@ -167,4 +167,30 @@
     <xacro:property name="sec_visual_parameter" value="${cfg_visual_parameter['visual_parameter']}" scope="parent" />
   </xacro:macro>
+  <!-- 从yaml文件中加载工具配置数据。 -->
+  <xacro:macro
+    name="read_tool_config"
+    params="physical_parameter_file
+            visual_parameter_file
+            force_abs_path">
+    <xacro:property name="force_abs_path" value="${force_abs_path}" scope="parent" />
+    <!-- 物理参数 -->
+    <xacro:property name="cfg_physical_parameter" value="${xacro.load_yaml(physical_parameter_file)}" />
+    <xacro:property name="sec_physical_parameter" value="${cfg_physical_parameter['physical_parameter']}" />
+    <xacro:property name="tool_mass" value="${sec_physical_parameter['tool']['mass']}" scope="parent" />
+    <xacro:property name="prop_tool_cog" value="${sec_physical_parameter['tool']['center_of_mass']}" scope="parent" />
+    <xacro:property name="tool_cog" value="${prop_tool_cog['x']} ${prop_tool_cog['y']} ${prop_tool_cog['z']}" scope="parent" />
+    <xacro:property name="prop_tool_inertia_rotation" value="${sec_physical_parameter['tool']['rotation']}" scope="parent" />
+    <xacro:property name="tool_inertia_rotation" value="${prop_tool_inertia_rotation['roll']} ${prop_tool_inertia_rotation['pitch']} ${prop_tool_inertia_rotation['yaw']}" scope="parent" />
+    <xacro:property name="prop_tool_inertia" value="${sec_physical_parameter['tool']['tensor']}" scope="parent" />
+    <xacro:property name="tool_inertia_ixx" value="${prop_tool_inertia['ixx']}" scope="parent" />
+    <xacro:property name="tool_inertia_ixy" value="${prop_tool_inertia['ixy']}" scope="parent" />
+    <xacro:property name="tool_inertia_ixz" value="${prop_tool_inertia['ixz']}" scope="parent" />
+    <xacro:property name="tool_inertia_iyy" value="${prop_tool_inertia['iyy']}" scope="parent" />
+    <xacro:property name="tool_inertia_iyz" value="${prop_tool_inertia['iyz']}" scope="parent" />
+    <xacro:property name="tool_inertia_izz" value="${prop_tool_inertia['izz']}" scope="parent" />
+    <!-- 视觉参数 -->
+    <xacro:property name="cfg_visual_parameter" value="${xacro.load_yaml(visual_parameter_file)}" />
+    <xacro:property name="sec_visual_parameter" value="${cfg_visual_parameter['visual_parameter']}" scope="parent" />
+  </xacro:macro>
   <!-- 根据指定的连杆名和模型类型返回模型文件参数，模型类型包括visual和collision，如果没有定义对应类型的参数，则返回空。 -->
   <xacro:macro name="get_mesh_param" params="name:=^ type:=^">

File: peeks_robot_descriptions/urdf/inc/create_robot.xacro (robot description, xacro)
@@ -14,5 +14,5 @@
             visual_parameter_file
             force_abs_path:=false">
-    <xacro:read_model_config
+    <xacro:read_robot_config
       joint_limit_parameter_file="${joint_limit_parameter_file}"
       robot_kinematics_parameter_file="${robot_kinematics_parameter_file}"
@@ -231,4 +231,5 @@
       </inertial>
     </link>
+    <link name="${tf_prefix}flange_link" />
     <!-- 关节 -->
     <joint name="${tf_prefix}base_joint" type="fixed">
@@ -321,4 +322,9 @@
       <dynamics damping="0" friction="0" />
     </joint>
+    <joint name="${tf_prefix}flange_joint" type="fixed">
+      <parent link="${tf_prefix}wrist_3_link" />
+      <child link="${tf_prefix}flange_link" />
+      <origin xyz="0 0 0" rpy="0 0 0" />
+    </joint>
   </xacro:macro>
 </robot>

File: peeks_robot_descriptions/urdf/robot.urdf.xacro (robot description, xacro)
@@ -3,11 +3,16 @@
   <xacro:arg name="robot_name" default="robot_1" />
   <xacro:arg name="robot_type" default="abb/crb15000" />
-  <xacro:arg name="tf_prefix" default="" />
   <xacro:arg name="joint_limit_param" default="$(find peeks_robot_descriptions)/config/robots/$(arg robot_type)/joint_limit.yaml" />
   <xacro:arg name="robot_kinematics_param" default="$(find peeks_robot_descriptions)/config/robots/$(arg robot_type)/robot_kinematics.yaml" />
-  <xacro:arg name="physical_param" default="$(find peeks_robot_descriptions)/config/robots/$(arg robot_type)/physical_parameter.yaml" />
-  <xacro:arg name="visual_param" default="$(find peeks_robot_descriptions)/config/robots/$(arg robot_type)/visual_parameter.yaml" />
+  <xacro:arg name="robot_physical_param" default="$(find peeks_robot_descriptions)/config/robots/$(arg robot_type)/physical_parameter.yaml" />
+  <xacro:arg name="robot_visual_param" default="$(find peeks_robot_descriptions)/config/robots/$(arg robot_type)/visual_parameter.yaml" />
+  <xacro:arg name="tool_name" default="tool_1" />
+  <xacro:arg name="tool_type" default="dummy" />
+  <xacro:arg name="tool_physical_param" default="$(find peeks_robot_descriptions)/config/tools/$(arg tool_type)/physical_parameter.yaml" />
+  <xacro:arg name="tool_visual_param" default="$(find peeks_robot_descriptions)/config/tools/$(arg tool_type)/visual_parameter.yaml" />
+  <xacro:arg name="tf_prefix" default="" />
   <xacro:arg name="force_abs_path" default="false" />
-  <xacro:include filename="$(find peeks_robot_descriptions)/urdf/robot_macro.xacro" />
+  <xacro:include filename="$(find peeks_robot_descriptions)/urdf/inc/create_robot.xacro" />
+  <xacro:include filename="$(find peeks_robot_descriptions)/urdf/inc/create_tool.xacro" />
   <link name="world_link" />
   <xacro:create_robot
@@ -17,8 +22,17 @@
     joint_limit_parameter_file="$(arg joint_limit_param)"
     robot_kinematics_parameter_file="$(arg robot_kinematics_param)"
-    physical_parameter_file="$(arg physical_param)"
-    visual_parameter_file="$(arg visual_param)"
+    physical_parameter_file="$(arg robot_physical_param)"
+    visual_parameter_file="$(arg robot_visual_param)"
     force_abs_path="$(arg force_abs_path)">
     <origin xyz="0 0 0" rpy="0 0 0" />
   </xacro:create_robot>
+  <xacro:create_tool
+    tool_name="$(arg tool_name)"
+    tf_prefix="$(arg tf_prefix)"
+    parent="$(arg tf_prefix)flange_link"
+    physical_parameter_file="$(arg tool_physical_param)"
+    visual_parameter_file="$(arg tool_visual_param)"
+    force_abs_path="$(arg force_abs_path)">
+    <origin xyz="0 0 0" rpy="0 0 0" />
+  </xacro:create_tool>
 </robot>

Commit message: fix: modify flange joint position

File: peeks_robot_descriptions/urdf/inc/common.xacro (robot description, xacro)
@@ -76,4 +76,10 @@
     <xacro:property name="wrist_3_pitch" value="${sec_robot_kinematics['wrist_3']['pitch']}" scope="parent" />
     <xacro:property name="wrist_3_yaw" value="${sec_robot_kinematics['wrist_3']['yaw']}" scope="parent" />
+    <xacro:property name="flange_x" value="${sec_robot_kinematics['flange']['x']}" scope="parent" />
+    <xacro:property name="flange_y" value="${sec_robot_kinematics['flange']['y']}" scope="parent" />
+    <xacro:property name="flange_z" value="${sec_robot_kinematics['flange']['z']}" scope="parent" />
+    <xacro:property name="flange_roll" value="${sec_robot_kinematics['flange']['roll']}" scope="parent" />
+    <xacro:property name="flange_pitch" value="${sec_robot_kinematics['flange']['pitch']}" scope="parent" />
+    <xacro:property name="flange_yaw" value="${sec_robot_kinematics['flange']['yaw']}" scope="parent" />
     <!-- 物理参数 -->
     <xacro:property name="cfg_physical_parameter" value="${xacro.load_yaml(physical_parameter_file)}" />

File: peeks_robot_descriptions/urdf/inc/create_robot.xacro (robot description, xacro)
@@ -325,5 +325,7 @@
       <parent link="${tf_prefix}wrist_3_link" />
       <child link="${tf_prefix}flange_link" />
-      <origin xyz="0 0 0" rpy="0 0 0" />
+      <origin
+        xyz="${flange_x} ${flange_y} ${flange_z}"
+        rpy="${flange_roll} ${flange_pitch} ${flange_yaw}" />
     </joint>
   </xacro:macro>

Commit message: refactor: modify the name of kinematics config file

File: peeks_robot_descriptions/urdf/inc/common.xacro (robot description, xacro)
@@ -5,5 +5,5 @@
     name="read_robot_config"
     params="joint_limit_parameter_file
-            robot_kinematics_parameter_file
+            default_kinematics_parameter_file
             physical_parameter_file
             visual_parameter_file
@@ -37,49 +37,49 @@
     <xacro:property name="wrist_3_velocity_limit" value="${sec_joint_limit['wrist_3']['max_velocity']}" scope="parent" />
     <xacro:property name="wrist_3_effort_limit" value="${sec_joint_limit['wrist_3']['max_effort']}" scope="parent" />
-    <!-- 机器人运动学参数 -->
-    <xacro:property name="cfg_robot_kinematics_parameter" value="${xacro.load_yaml(robot_kinematics_parameter_file)}" />
-    <xacro:property name="sec_robot_kinematics" value="${cfg_robot_kinematics_parameter['robot_kinematics']}" />
-    <xacro:property name="shoulder_x" value="${sec_robot_kinematics['shoulder']['x']}" scope="parent" />
-    <xacro:property name="shoulder_y" value="${sec_robot_kinematics['shoulder']['y']}" scope="parent" />
-    <xacro:property name="shoulder_z" value="${sec_robot_kinematics['shoulder']['z']}" scope="parent" />
-    <xacro:property name="shoulder_roll" value="${sec_robot_kinematics['shoulder']['roll']}" scope="parent" />
-    <xacro:property name="shoulder_pitch" value="${sec_robot_kinematics['shoulder']['pitch']}" scope="parent" />
-    <xacro:property name="shoulder_yaw" value="${sec_robot_kinematics['shoulder']['yaw']}" scope="parent" />
-    <xacro:property name="upper_arm_x" value="${sec_robot_kinematics['upper_arm']['x']}" scope="parent" />
-    <xacro:property name="upper_arm_y" value="${sec_robot_kinematics['upper_arm']['y']}" scope="parent" />
-    <xacro:property name="upper_arm_z" value="${sec_robot_kinematics['upper_arm']['z']}" scope="parent" />
-    <xacro:property name="upper_arm_roll" value="${sec_robot_kinematics['upper_arm']['roll']}" scope="parent" />
-    <xacro:property name="upper_arm_pitch" value="${sec_robot_kinematics['upper_arm']['pitch']}" scope="parent" />
-    <xacro:property name="upper_arm_yaw" value="${sec_robot_kinematics['upper_arm']['yaw']}" scope="parent" />
-    <xacro:property name="forearm_x" value="${sec_robot_kinematics['forearm']['x']}" scope="parent" />
-    <xacro:property name="forearm_y" value="${sec_robot_kinematics['forearm']['y']}" scope="parent" />
-    <xacro:property name="forearm_z" value="${sec_robot_kinematics['forearm']['z']}" scope="parent" />
-    <xacro:property name="forearm_roll" value="${sec_robot_kinematics['forearm']['roll']}" scope="parent" />
-    <xacro:property name="forearm_pitch" value="${sec_robot_kinematics['forearm']['pitch']}" scope="parent" />
-    <xacro:property name="forearm_yaw" value="${sec_robot_kinematics['forearm']['yaw']}" scope="parent" />
-    <xacro:property name="wrist_1_x" value="${sec_robot_kinematics['wrist_1']['x']}" scope="parent" />
-    <xacro:property name="wrist_1_y" value="${sec_robot_kinematics['wrist_1']['y']}" scope="parent" />
-    <xacro:property name="wrist_1_z" value="${sec_robot_kinematics['wrist_1']['z']}" scope="parent" />
-    <xacro:property name="wrist_1_roll" value="${sec_robot_kinematics['wrist_1']['roll']}" scope="parent" />
-    <xacro:property name="wrist_1_pitch" value="${sec_robot_kinematics['wrist_1']['pitch']}" scope="parent" />
-    <xacro:property name="wrist_1_yaw" value="${sec_robot_kinematics['wrist_1']['yaw']}" scope="parent" />
-    <xacro:property name="wrist_2_x" value="${sec_robot_kinematics['wrist_2']['x']}" scope="parent" />
-    <xacro:property name="wrist_2_y" value="${sec_robot_kinematics['wrist_2']['y']}" scope="parent" />
-    <xacro:property name="wrist_2_z" value="${sec_robot_kinematics['wrist_2']['z']}" scope="parent" />
-    <xacro:property name="wrist_2_roll" value="${sec_robot_kinematics['wrist_2']['roll']}" scope="parent" />
-    <xacro:property name="wrist_2_pitch" value="${sec_robot_kinematics['wrist_2']['pitch']}" scope="parent" />
-    <xacro:property name="wrist_2_yaw" value="${sec_robot_kinematics['wrist_2']['yaw']}" scope="parent" />
-    <xacro:property name="wrist_3_x" value="${sec_robot_kinematics['wrist_3']['x']}" scope="parent" />
-    <xacro:property name="wrist_3_y" value="${sec_robot_kinematics['wrist_3']['y']}" scope="parent" />
-    <xacro:property name="wrist_3_z" value="${sec_robot_kinematics['wrist_3']['z']}" scope="parent" />
-    <xacro:property name="wrist_3_roll" value="${sec_robot_kinematics['wrist_3']['roll']}" scope="parent" />
-    <xacro:property name="wrist_3_pitch" value="${sec_robot_kinematics['wrist_3']['pitch']}" scope="parent" />
-    <xacro:property name="wrist_3_yaw" value="${sec_robot_kinematics['wrist_3']['yaw']}" scope="parent" />
-    <xacro:property name="flange_x" value="${sec_robot_kinematics['flange']['x']}" scope="parent" />
-    <xacro:property name="flange_y" value="${sec_robot_kinematics['flange']['y']}" scope="parent" />
-    <xacro:property name="flange_z" value="${sec_robot_kinematics['flange']['z']}" scope="parent" />
-    <xacro:property name="flange_roll" value="${sec_robot_kinematics['flange']['roll']}" scope="parent" />
-    <xacro:property name="flange_pitch" value="${sec_robot_kinematics['flange']['pitch']}" scope="parent" />
-    <xacro:property name="flange_yaw" value="${sec_robot_kinematics['flange']['yaw']}" scope="parent" />
+    <!-- 默认运动学参数 -->
+    <xacro:property name="cfg_default_kinematics_parameter" value="${xacro.load_yaml(default_kinematics_parameter_file)}" />
+    <xacro:property name="sec_default_kinematics" value="${cfg_default_kinematics_parameter['default_kinematics']}" />
+    <xacro:property name="shoulder_x" value="${sec_default_kinematics['shoulder']['x']}" scope="parent" />
+    <xacro:property name="shoulder_y" value="${sec_default_kinematics['shoulder']['y']}" scope="parent" />
+    <xacro:property name="shoulder_z" value="${sec_default_kinematics['shoulder']['z']}" scope="parent" />
+    <xacro:property name="shoulder_roll" value="${sec_default_kinematics['shoulder']['roll']}" scope="parent" />
+    <xacro:property name="shoulder_pitch" value="${sec_default_kinematics['shoulder']['pitch']}" scope="parent" />
+    <xacro:property name="shoulder_yaw" value="${sec_default_kinematics['shoulder']['yaw']}" scope="parent" />
+    <xacro:property name="upper_arm_x" value="${sec_default_kinematics['upper_arm']['x']}" scope="parent" />
+    <xacro:property name="upper_arm_y" value="${sec_default_kinematics['upper_arm']['y']}" scope="parent" />
+    <xacro:property name="upper_arm_z" value="${sec_default_kinematics['upper_arm']['z']}" scope="parent" />
+    <xacro:property name="upper_arm_roll" value="${sec_default_kinematics['upper_arm']['roll']}" scope="parent" />
+    <xacro:property name="upper_arm_pitch" value="${sec_default_kinematics['upper_arm']['pitch']}" scope="parent" />
+    <xacro:property name="upper_arm_yaw" value="${sec_default_kinematics['upper_arm']['yaw']}" scope="parent" />
+    <xacro:property name="forearm_x" value="${sec_default_kinematics['forearm']['x']}" scope="parent" />
+    <xacro:property name="forearm_y" value="${sec_default_kinematics['forearm']['y']}" scope="parent" />
+    <xacro:property name="forearm_z" value="${sec_default_kinematics['forearm']['z']}" scope="parent" />
+    <xacro:property name="forearm_roll" value="${sec_default_kinematics['forearm']['roll']}" scope="parent" />
+    <xacro:property name="forearm_pitch" value="${sec_default_kinematics['forearm']['pitch']}" scope="parent" />
+    <xacro:property name="forearm_yaw" value="${sec_default_kinematics['forearm']['yaw']}" scope="parent" />
+    <xacro:property name="wrist_1_x" value="${sec_default_kinematics['wrist_1']['x']}" scope="parent" />
+    <xacro:property name="wrist_1_y" value="${sec_default_kinematics['wrist_1']['y']}" scope="parent" />
+    <xacro:property name="wrist_1_z" value="${sec_default_kinematics['wrist_1']['z']}" scope="parent" />
+    <xacro:property name="wrist_1_roll" value="${sec_default_kinematics['wrist_1']['roll']}" scope="parent" />
+    <xacro:property name="wrist_1_pitch" value="${sec_default_kinematics['wrist_1']['pitch']}" scope="parent" />
+    <xacro:property name="wrist_1_yaw" value="${sec_default_kinematics['wrist_1']['yaw']}" scope="parent" />
+    <xacro:property name="wrist_2_x" value="${sec_default_kinematics['wrist_2']['x']}" scope="parent" />
+    <xacro:property name="wrist_2_y" value="${sec_default_kinematics['wrist_2']['y']}" scope="parent" />
+    <xacro:property name="wrist_2_z" value="${sec_default_kinematics['wrist_2']['z']}" scope="parent" />
+    <xacro:property name="wrist_2_roll" value="${sec_default_kinematics['wrist_2']['roll']}" scope="parent" />
+    <xacro:property name="wrist_2_pitch" value="${sec_default_kinematics['wrist_2']['pitch']}" scope="parent" />
+    <xacro:property name="wrist_2_yaw" value="${sec_default_kinematics['wrist_2']['yaw']}" scope="parent" />
+    <xacro:property name="wrist_3_x" value="${sec_default_kinematics['wrist_3']['x']}" scope="parent" />
+    <xacro:property name="wrist_3_y" value="${sec_default_kinematics['wrist_3']['y']}" scope="parent" />
+    <xacro:property name="wrist_3_z" value="${sec_default_kinematics['wrist_3']['z']}" scope="parent" />
+    <xacro:property name="wrist_3_roll" value="${sec_default_kinematics['wrist_3']['roll']}" scope="parent" />
+    <xacro:property name="wrist_3_pitch" value="${sec_default_kinematics['wrist_3']['pitch']}" scope="parent" />
+    <xacro:property name="wrist_3_yaw" value="${sec_default_kinematics['wrist_3']['yaw']}" scope="parent" />
+    <xacro:property name="flange_x" value="${sec_default_kinematics['flange']['x']}" scope="parent" />
+    <xacro:property name="flange_y" value="${sec_default_kinematics['flange']['y']}" scope="parent" />
+    <xacro:property name="flange_z" value="${sec_default_kinematics['flange']['z']}" scope="parent" />
+    <xacro:property name="flange_roll" value="${sec_default_kinematics['flange']['roll']}" scope="parent" />
+    <xacro:property name="flange_pitch" value="${sec_default_kinematics['flange']['pitch']}" scope="parent" />
+    <xacro:property name="flange_yaw" value="${sec_default_kinematics['flange']['yaw']}" scope="parent" />
     <!-- 物理参数 -->
     <xacro:property name="cfg_physical_parameter" value="${xacro.load_yaml(physical_parameter_file)}" />

File: peeks_robot_descriptions/urdf/inc/create_robot.xacro (robot description, xacro)
@@ -10,5 +10,5 @@
             *origin
             joint_limit_parameter_file
-            robot_kinematics_parameter_file
+            default_kinematics_parameter_file
             physical_parameter_file
             visual_parameter_file
@@ -16,5 +16,5 @@
     <xacro:read_robot_config
       joint_limit_parameter_file="${joint_limit_parameter_file}"
-      robot_kinematics_parameter_file="${robot_kinematics_parameter_file}"
+      default_kinematics_parameter_file="${default_kinematics_parameter_file}"
       physical_parameter_file="${physical_parameter_file}"
       visual_parameter_file="${visual_parameter_file}"

File: peeks_robot_descriptions/urdf/robot.urdf.xacro (robot description, xacro)
@@ -3,6 +3,6 @@
   <xacro:arg name="robot_name" default="robot_1" />
   <xacro:arg name="robot_type" default="abb/crb15000" />
-  <xacro:arg name="joint_limit_param" default="$(find peeks_robot_descriptions)/config/robots/$(arg robot_type)/joint_limit.yaml" />
-  <xacro:arg name="robot_kinematics_param" default="$(find peeks_robot_descriptions)/config/robots/$(arg robot_type)/robot_kinematics.yaml" />
+  <xacro:arg name="robot_joint_limit_param" default="$(find peeks_robot_descriptions)/config/robots/$(arg robot_type)/joint_limit.yaml" />
+  <xacro:arg name="robot_default_kinematics_param" default="$(find peeks_robot_descriptions)/config/robots/$(arg robot_type)/default_kinematics.yaml" />
   <xacro:arg name="robot_physical_param" default="$(find peeks_robot_descriptions)/config/robots/$(arg robot_type)/physical_parameter.yaml" />
   <xacro:arg name="robot_visual_param" default="$(find peeks_robot_descriptions)/config/robots/$(arg robot_type)/visual_parameter.yaml" />
@@ -20,6 +20,6 @@
     tf_prefix="$(arg tf_prefix)"
     parent="world_link"
-    joint_limit_parameter_file="$(arg joint_limit_param)"
-    robot_kinematics_parameter_file="$(arg robot_kinematics_param)"
+    joint_limit_parameter_file="$(arg robot_joint_limit_param)"
+    default_kinematics_parameter_file="$(arg robot_default_kinematics_param)"
     physical_parameter_file="$(arg robot_physical_param)"
     visual_parameter_file="$(arg robot_visual_param)"
